File: Taller1/Taller1.kicad_sch (KiCad schematic)
At the start: 9 parts, among them U1 DHT11, U2 Sensor de luz, U3 HL-69, U4 SX1262-XIAO

Commit message: Ultima versao de KiCad
Parts:
- removed U2: Sensor de luz, Sensor_Pressure:CFSensor_XGZP6859D_7x7mm, symbol Sensor_Pressure:XGZP6859D
- removed U3: HL-69, Sensor_Pressure:CFSensor_XGZP6859D_7x7mm, symbol Sensor_Pressure:XGZP6859D
- LM393-HL69, LM393-LDR1: footprint (none) -> Connector_PinHeader_2.54mm:PinHeader_1x04_P2.54mm_Vertical
- R1: footprint (none) -> Resistor_SMD:R_0805_2012Metric
Other:
- moved on the sheet: LM393-HL69, LM393-LDR1, U4

Commit message: ultima version PCB
Parts:
- removed R1: 4,7k, Resistor_SMD:R_0805_2012Metric, symbol Device:R_US
- added DHT1, DHT11: Conn_01x03, Connector_PinHeader_2.54mm:PinHeader_1x03_P2.54mm_Vertical, symbol Connector_Generic:Conn_01x03
- added R2: 4700, Resistor_THT:R_Axial_DIN0207_L6.3mm_D2.5mm_P7.62mm_Horizontal, symbol Device:R_US
Connections:
- net Alimentacion 3.3v: now also DHT11.1 (Pin_1); no longer U1.1 (VDD)
- net GND: now also DHT11.3 (Pin_3); no longer U1.4 (GND)
- net GPIO1: now also U4.9 (DIO1); no longer U4.10 (RST)
- net GPIO3: now also U4.10 (RST); no longer U4.9 (DIO1)
- net GNDA: now reaches CIAA-P1-1.7 (GNDA)
- net at U1.2 (DATA): now also R2.2
- net GPIO5: now reaches CIAA-P2-1.36 (GPIO5)
- net GPIO5: now also U4.12 (NSS)
- net GPIO7: now reaches CIAA-P2-1.38 (GPIO7)
- net GPIO7: now also DHT11.2 (Pin_2)
- net GPIO0: no longer names the net of CIAA-P2-1.29 (GPIO0)
- net GPIO2: no longer names the net of CIAA-P2-1.31 (GPIO2)
- net GPIO2: no longer U4.12 (NSS)
- new net: R2.1, U1.1 (VDD)
